File: Hardware/MicroMod_CAN-Bus_Function_Board.brd (EAGLE design)
At the start: 38 x 65 mm, 92 parts, among them J1 MICROMOD_FUNCTION_STANDARD, Q1 220mA/50V/3.5Ω, U1 XC9140, U2 MCP2515, U3 TXS0108, U4 MCP2551, X1 DB9 Plug, Y1 16MHz

Commit message: x03
Connections:
- net GND: now also J1.2, J1.8
- net MM_RXCAN: now also J1.43, TP1.1; no longer J1.41, TP2.1
- net MM_TXCAN: now also J1.41, TP2.1; no longer J1.43, TP1.1
Routing:
- net GND: track 16.7 -> 20.5 mm
- net MM_TXCAN: track 10.9 -> 11.9 mm
- net MM_RXCAN: track 10.9 -> 10.7 mm, vias 0 -> 2
Other:
- board text added: "x03"
- board text removed: "x02"
Changed lines of the file:
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@@
 <drawing>
 <settings>
-<setting alwaysvectorfont="yes"/>
+<setting alwaysvectorfont="no"/>
 <setting verticaltext="up"/>
 </settings>
@@
 <vertex x="16.891" y="23.622"/>
 </polygon>
-<text x="4.318" y="4.191" size="1.778" layer="16" font="vector" ratio="15" rot="MR0">x02</text>
+<text x="4.318" y="4.191" size="1.778" layer="16" font="vector" ratio="15" rot="MR0">x03</text>
 </plain>
 <attributes>
@@
 <wire x1="20.3" y1="2.941" x2="19.431" y2="3.81" width="0.254" layer="1"/>
 <wire x1="17.3" y1="1.275" x2="17.3" y2="2.639" width="0.254" layer="1"/>
-<wire x1="17.3" y1="2.639" x2="16.383" y2="3.556" width="0.254" layer="1"/>
-<via x="16.383" y="3.556" extent="1-16" drill="0.3048"/>
+<wire x1="17.3" y1="2.639" x2="16.637" y2="3.302" width="0.254" layer="1"/>
+<via x="16.637" y="3.302" extent="1-16" drill="0.3048"/>
 <wire x1="9.8" y1="1.275" x2="9.8" y2="4.17" width="0.254" layer="1"/>
 <wire x1="9.8" y1="4.17" x2="8.89" y2="5.08" width="0.254" layer="1"/>
@@
 <via x="26.543" y="50.546" extent="1-16" drill="0.3048"/>
 <via x="29.083" y="50.546" extent="1-16" drill="0.3048"/>
+<contactref element="J1" pad="2"/>
+<contactref element="J1" pad="8"/>
+<wire x1="28.05" y1="1.525" x2="28.05" y2="3.285" width="0.1524" layer="16"/>
+<wire x1="28.05" y1="3.285" x2="28.067" y2="3.302" width="0.1524" layer="16"/>
+<wire x1="26.55" y1="1.525" x2="26.55" y2="3.69" width="0.1524" layer="16"/>
+<wire x1="26.55" y1="3.69" x2="26.67" y2="3.81" width="0.1524" layer="16"/>
 <wire x1="37.05" y1="41.9" x2="35.75" y2="44" width="0" layer="19" extent="1-1"/>
 <wire x1="2.35" y1="44" x2="1.05" y2="41.9" width="0" layer="19" extent="1-1"/>
 </signal>
 <signal name="MM_TXCAN">
+<contactref element="U3" pad="5"/>
+<wire x1="12.45" y1="9.63" x2="12.45" y2="7.235" width="0.1524" layer="1"/>
+<contactref element="J1" pad="41"/>
+<contactref element="TP2" pad="1"/>
+<wire x1="12.45" y1="7.235" x2="13.589" y2="6.096" width="0.1524" layer="1"/>
+<wire x1="15.494" y1="6.096" x2="16.51" y2="5.08" width="0.1524" layer="1"/>
+<wire x1="13.589" y1="6.096" x2="15.494" y2="6.096" width="0.1524" layer="1"/>
+<wire x1="16.51" y1="5.08" x2="18.3" y2="3.29" width="0.1524" layer="1"/>
+<wire x1="18.3" y1="3.29" x2="18.3" y2="1.275" width="0.1524" layer="1"/>
+</signal>
+<signal name="MM_RXCAN">
+<contactref element="U3" pad="6"/>
 <contactref element="J1" pad="43"/>
 <contactref element="TP1" pad="1"/>
-<contactref element="U3" pad="5"/>
-<wire x1="15.24" y1="5.08" x2="12.45" y2="7.87" width="0.1524" layer="1"/>
-<wire x1="12.45" y1="7.87" x2="12.45" y2="9.63" width="0.1524" layer="1"/>
-<wire x1="17.8" y1="3.028" x2="16.51" y2="4.318" width="0.1524" layer="1"/>
-<wire x1="16.51" y1="4.318" x2="16.002" y2="4.318" width="0.1524" layer="1"/>
-<wire x1="16.002" y1="4.318" x2="15.24" y2="5.08" width="0.1524" layer="1"/>
-<wire x1="17.8" y1="1.275" x2="17.8" y2="3.028" width="0.1524" layer="1"/>
-</signal>
-<signal name="MM_RXCAN">
-<contactref element="J1" pad="41"/>
-<contactref element="TP2" pad="1"/>
-<contactref element="U3" pad="6"/>
-<wire x1="18.3" y1="1.275" x2="18.3" y2="3.29" width="0.1524" layer="1"/>
-<wire x1="18.3" y1="3.29" x2="16.51" y2="5.08" width="0.1524" layer="1"/>
-<wire x1="16.51" y1="5.08" x2="15.494" y2="6.096" width="0.1524" layer="1"/>
-<wire x1="15.494" y1="6.096" x2="14.859" y2="6.096" width="0.1524" layer="1"/>
-<wire x1="14.859" y1="6.096" x2="12.95" y2="8.005" width="0.1524" layer="1"/>
-<wire x1="12.95" y1="8.005" x2="12.95" y2="9.63" width="0.1524" layer="1"/>
+<wire x1="12.95" y1="7.751" x2="13.589" y2="7.112" width="0.1524" layer="1"/>
+<via x="13.589" y="7.112" extent="1-16" drill="0.3048"/>
+<wire x1="13.589" y1="7.112" x2="15.24" y2="5.461" width="0.1524" layer="16"/>
+<wire x1="15.24" y1="5.461" x2="15.24" y2="5.08" width="0.1524" layer="16"/>
+<via x="15.24" y="5.08" extent="1-16" drill="0.3048"/>
+<wire x1="15.24" y1="5.08" x2="16.51" y2="3.81" width="0.1524" layer="1"/>
+<wire x1="16.51" y1="3.81" x2="17.145" y2="3.81" width="0.1524" layer="1"/>
+<wire x1="17.145" y1="3.81" x2="17.8" y2="3.155" width="0.1524" layer="1"/>
+<wire x1="17.8" y1="3.155" x2="17.8" y2="1.275" width="0.1524" layer="1"/>
+<wire x1="12.95" y1="9.63" x2="12.95" y2="7.751" width="0.1524" layer="1"/>
 </signal>
 <signal name="MM_SDI">
@@
 <wire x1="36.195" y1="8.255" x2="34.29" y2="6.35" width="0.1524" layer="1"/>
 <via x="34.29" y="6.35" extent="1-16" drill="0.3048"/>
-<wire x1="34.29" y1="6.35" x2="16.51" y2="6.35" width="0.1524" layer="16"/>
-<wire x1="16.51" y1="6.35" x2="13.97" y2="3.81" width="0.1524" layer="16"/>
 <via x="13.97" y="3.81" extent="1-16" drill="0.3048"/>
 <wire x1="13.97" y1="3.81" x2="15.8" y2="1.98" width="0.1524" layer="1"/>
 <wire x1="15.8" y1="1.98" x2="15.8" y2="1.275" width="0.1524" layer="1"/>
+<wire x1="20.32" y1="6.35" x2="17.78" y2="3.81" width="0.1524" layer="16"/>
+<wire x1="34.29" y1="6.35" x2="20.32" y2="6.35" width="0.1524" layer="16"/>
+<wire x1="17.78" y1="3.81" x2="13.97" y2="3.81" width="0.1524" layer="16"/>
 </signal>
 <signal name="N$11">

Commit message: Housekeeping
Parts:
- added LOGO2: SPECIAL_INSTRUCTIONS-ORDERING, SparkFun-Aesthetics:ORDERING_INSTRUCTIONS
- U$39: device SparkFun-Aesthetics:SFE_LOGO_NAME_FLAME_10MM -> SparkX:SPARKX-MEDIUM
- U$4: device SparkFun-Aesthetics:SFE_LOGO_NAME_FLAME_.1 -> SparkX:SPARKX-MEDIUM
- moved U$1 31.6 mm to (2.67, 7.24)
- moved U$2 31.4 mm to (1.40, 10.0)
- moved U$3 31.4 mm to (3.94, 10.0)
- moved U$4 21.8 mm to (2.54, 33.0)
- moved U$39 19.1 mm to (19.1, 14.0)
Other:
- board text added: "2-Layer"
- board text added: "Beveled Edge"
- board text added: "Board Thickness is 0.8mm"
- board text added: "ENIG Finish"
- board text added: "Nick P"
Changed lines of the file:
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@@
 <layers>
 <layer number="1" name="Top" color="4" fill="1" visible="yes" active="yes"/>
-<layer number="2" name="Route2" color="16" fill="1" visible="no" active="yes"/>
+<layer number="2" name="Route2" color="16" fill="1" visible="yes" active="yes"/>
 <layer number="3" name="Route3" color="17" fill="1" visible="no" active="no"/>
 <layer number="4" name="Route4" color="18" fill="1" visible="no" active="no"/>
@@
 <layer number="13" name="Route13" color="21" fill="1" visible="no" active="no"/>
 <layer number="14" name="Route14" color="22" fill="1" visible="no" active="no"/>
-<layer number="15" name="Route15" color="23" fill="1" visible="no" active="yes"/>
+<layer number="15" name="Route15" color="23" fill="1" visible="yes" active="yes"/>
 <layer number="16" name="Bottom" color="1" fill="1" visible="yes" active="yes"/>
 <layer number="17" name="Pads" color="2" fill="1" visible="yes" active="yes"/>
@@
 <layer number="44" name="Drills" color="7" fill="1" visible="no" active="yes"/>
 <layer number="45" name="Holes" color="7" fill="1" visible="yes" active="yes"/>
-<layer number="46" name="Milling" color="3" fill="1" visible="no" active="yes"/>
+<layer number="46" name="Milling" color="3" fill="1" visible="yes" active="yes"/>
 <layer number="47" name="Measures" color="7" fill="1" visible="no" active="yes"/>
 <layer number="48" name="Document" color="7" fill="1" visible="no" active="yes"/>
@@
 </polygon>
 <text x="4.318" y="4.191" size="1.778" layer="16" font="vector" ratio="15" rot="MR0">x03</text>
+<text x="22.86" y="-11.43" size="1.778" layer="51" font="vector" ratio="15">Nick P</text>
+<text x="41.63" y="52.03" size="1.778" layer="51" font="vector" ratio="15">Board Thickness is 0.8mm</text>
+<text x="41.63" y="49.49" size="1.778" layer="51" font="vector" ratio="15">2-Layer</text>
+<text x="41.63" y="46.95" size="1.778" layer="51" font="vector" ratio="15">Beveled Edge</text>
+<text x="41.63" y="44.41" size="1.778" layer="51" font="vector" ratio="15">ENIG Finish</text>
 </plain>
 <attributes>
@@
 <attribute name="VALUE" x="24.13" y="25.908" size="0.6096" layer="27" font="vector" ratio="20" align="top-center"/>
 </element>
-<element name="U$1" library="SparkFun-MicroMod" package="MICROMOD_MI_LOGO_1" value="" x="19.177" y="34.163" smashed="yes" rot="R90"/>
-<element name="U$2" library="output" package="FUNCTION0" value="" x="17.907" y="36.703" smashed="yes" rot="R90"/>
-<element name="U$3" library="output" package="CAN_BUS0" value="" x="20.447" y="36.703" smashed="yes" rot="R90"/>
+<element name="U$1" library="SparkFun-MicroMod" package="MICROMOD_MI_LOGO_1" value="" x="2.667" y="7.239" smashed="yes" rot="R90"/>
+<element name="U$2" library="output" package="FUNCTION0" value="" x="1.397" y="10.033" smashed="yes" rot="R90"/>
+<element name="U$3" library="output" package="CAN_BUS0" value="" x="3.937" y="10.033" smashed="yes" rot="R90"/>
 <element name="U$17" library="output" package="GND0" value="" x="14.986" y="43.561" smashed="yes" rot="MR0"/>
 <element name="U$19" library="output" package="OBD#II0" value="" x="6.096" y="49.276" smashed="yes" rot="MR0"/>
@@
 <element name="U$24" library="output" package="PIN_30" value="" x="10.287" y="43.561" smashed="yes" rot="MR0"/>
 <element name="U$25" library="output" package="PIN_50" value="" x="6.35" y="45.466" smashed="yes" rot="MR0"/>
-<element name="U$4" library="SparkFun-Aesthetics" package="SFE_LOGO_NAME_FLAME_.1" value="" x="5.461" y="11.43" smashed="yes" rot="R90"/>
 <element name="U$5" library="output" package="#CANH_#0" value="" x="36.195" y="53.34" smashed="yes" rot="R90"/>
 <element name="U$6" library="output" package="#CANL_#0" value="" x="33.655" y="53.467" smashed="yes" rot="R90"/>
@@
 <element name="U$37" library="output" package="CAN_BUS0" value="" x="22.987" y="7.493" smashed="yes" rot="MR0"/>
 <element name="U$38" library="output" package="FUNCTION0" value="" x="22.987" y="10.033" smashed="yes" rot="MR0"/>
-<element name="U$39" library="SparkFun-Aesthetics" package="SFE_LOGO_NAME_FLAME_10MM" value="" x="19.05" y="33.02" smashed="yes" rot="MR0"/>
 <element name="U$40" library="SparkFun-Aesthetics" package="OSHW-LOGO-S" value="" x="2.54" y="6.35" smashed="yes" rot="MR0"/>
 <element name="FD1" library="SparkFun-Aesthetics" package="FIDUCIAL-1X2" value="FIDUCIAL1X2" x="1.27" y="63.5" smashed="yes"/>
 <element name="FD2" library="SparkFun-Aesthetics" package="FIDUCIAL-1X2" value="FIDUCIAL1X2" x="36.83" y="5.08" smashed="yes"/>
 <element name="FD3" library="SparkFun-Aesthetics" package="FIDUCIAL-0.2MM" value="FIDUCIAL0.2MM" x="1.27" y="5.08" smashed="yes"/>
+<element name="U$4" library="SparkX" package="SPARKX-MEDIUM" value="" x="2.54" y="33.02" smashed="yes" rot="R90"/>
+<element name="U$39" library="SparkX" package="SPARKX-MEDIUM" value="" x="19.05" y="13.97" smashed="yes" rot="MR0"/>
+<element name="LOGO2" library="SparkFun-Aesthetics" package="ORDERING_INSTRUCTIONS" value="SPECIAL_INSTRUCTIONS-ORDERING" x="40.36" y="64.73" smashed="yes"/>
 </elements>
 <signals>
@@
 <via x="13.335" y="47.371" extent="1-16" drill="0.3048"/>
 <wire x1="13.335" y1="47.371" x2="20.32" y2="47.371" width="0.1524" layer="16"/>
-<wire x1="20.32" y1="47.371" x2="27.94" y2="47.371" width="0.1524" layer="16"/>
-<wire x1="28.321" y1="47.371" x2="28.448" y2="47.371" width="0.1524" layer="16"/>
-<wire x1="28.448" y1="47.371" x2="31.75" y2="47.371" width="0.1524" layer="16"/>
+<wire x1="20.32" y1="47.371" x2="28.321" y2="47.371" width="0.1524" layer="16"/>
+<wire x1="28.321" y1="47.371" x2="31.75" y2="47.371" width="0.1524" layer="16"/>
 <wire x1="31.75" y1="47.371" x2="33.655" y2="49.276" width="0.1524" layer="16"/>
 <via x="33.655" y="49.276" extent="1-16" drill="0.3048"/>
@@
 <wire x1="28.3464" y1="45.72" x2="28.3464" y2="47.3456" width="0.1524" layer="16"/>
 <wire x1="28.3464" y1="47.3456" x2="28.321" y2="47.371" width="0.1524" layer="16"/>
-<wire x1="27.94" y1="47.371" x2="28.321" y2="47.371" width="0.1524" layer="16"/>
 </signal>
 <signal name="N$9">
