File: Hardware/MicroMod_CAN-Bus_Function_Board.sch (EAGLE design)
At the start: 52 parts, among them J1 MICROMOD_FUNCTION_STANDARD, Q1 220mA/50V/3.5Ω, U1 XC9140, U2 MCP2515, U3 TXS0108, U4 MCP2551, X1 DB9 Plug, Y1 16MHz

Commit message: x03
Connections:
- net MM_RXCAN: now also TP1.1; no longer TP2.1
- net MM_TXCAN: now also TP2.1; no longer TP1.1
Other:
- moved on the sheet: TP1, TP2
Changed lines of the file:
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@@
 <drawing>
 <settings>
-<setting alwaysvectorfont="yes"/>
+<setting alwaysvectorfont="no"/>
 <setting verticaltext="up"/>
 </settings>
@@
 <instance part="J1" gate="J1" x="35.56" y="142.24" smashed="yes">
 <attribute name="NAME" x="20.32" y="170.688" size="1.778" layer="95"/>
-<attribute name="VALUE" x="20.32" y="106.68" size="1.778" layer="96"/>
+<attribute name="VALUE" x="20.32" y="104.14" size="1.778" layer="96"/>
 </instance>
 <instance part="J2" gate="G$1" x="137.16" y="50.8" smashed="yes" rot="R180">
@@
 <attribute name="VALUE" x="15.24" y="172.974" size="1.778" layer="96" align="bottom-center"/>
 </instance>
-<instance part="GND1" gate="1" x="15.24" y="106.68" smashed="yes">
-<attribute name="VALUE" x="15.24" y="106.426" size="1.778" layer="96" align="top-center"/>
+<instance part="GND1" gate="1" x="15.24" y="104.14" smashed="yes">
+<attribute name="VALUE" x="15.24" y="103.886" size="1.778" layer="96" align="top-center"/>
 </instance>
 <instance part="U2" gate="&gt;NAME" x="111.76" y="154.94" smashed="yes">
@@
 <attribute name="VALUE" x="137.16" y="122.174" size="1.778" layer="96" font="vector" align="bottom-center"/>
 </instance>
-<instance part="TP1" gate="G$1" x="15.24" y="139.7" smashed="yes" rot="R90">
-<attribute name="NAME" x="12.7" y="144.78" size="1.778" layer="95" font="vector" rot="R180"/>
-</instance>
-<instance part="TP2" gate="G$1" x="15.24" y="137.16" smashed="yes" rot="R270">
-<attribute name="NAME" x="12.7" y="134.62" size="1.778" layer="95" font="vector" rot="R180"/>
+<instance part="TP1" gate="G$1" x="15.24" y="132.08" smashed="yes" rot="R90">
+<attribute name="NAME" x="12.7" y="137.16" size="1.778" layer="95" font="vector" rot="R180"/>
+</instance>
+<instance part="TP2" gate="G$1" x="15.24" y="124.46" smashed="yes" rot="R270">
+<attribute name="NAME" x="12.7" y="121.92" size="1.778" layer="95" font="vector" rot="R180"/>
 </instance>
 <instance part="TP3" gate="G$1" x="167.64" y="144.78" smashed="yes" rot="R270">
@@
 <net name="MM_TXCAN" class="0">
 <segment>
-<pinref part="J1" gate="J1" pin="CAN-TX"/>
-<wire x1="17.78" y1="139.7" x2="15.24" y2="139.7" width="0.1524" layer="91"/>
-<label x="12.7" y="139.7" size="1.27" layer="95" rot="R180" xref="yes"/>
-<pinref part="TP1" gate="G$1" pin="1"/>
-<wire x1="15.24" y1="139.7" x2="12.7" y2="139.7" width="0.1524" layer="91"/>
-<junction x="15.24" y="139.7"/>
-</segment>
-<segment>
 <wire x1="22.86" y1="66.04" x2="17.78" y2="66.04" width="0.1524" layer="91"/>
 <label x="17.78" y="66.04" size="1.27" layer="95" rot="R180" xref="yes"/>
 <pinref part="U3" gate="G$1" pin="A4"/>
 </segment>
+<segment>
+<pinref part="J1" gate="J1" pin="CAN-TX"/>
+<wire x1="17.78" y1="127" x2="15.24" y2="127" width="0.1524" layer="91"/>
+<label x="12.7" y="127" size="1.27" layer="95" rot="R180" xref="yes"/>
+<pinref part="TP2" gate="G$1" pin="1"/>
+<wire x1="15.24" y1="127" x2="12.7" y2="127" width="0.1524" layer="91"/>
+<wire x1="15.24" y1="127" x2="15.24" y2="124.46" width="0.1524" layer="91"/>
+<junction x="15.24" y="127"/>
+</segment>
 </net>
 <net name="MM_RXCAN" class="0">
-<segment>
-<pinref part="J1" gate="J1" pin="CAN-RX"/>
-<wire x1="17.78" y1="137.16" x2="15.24" y2="137.16" width="0.1524" layer="91"/>
-<label x="12.7" y="137.16" size="1.27" layer="95" rot="R180" xref="yes"/>
-<pinref part="TP2" gate="G$1" pin="1"/>
-<wire x1="15.24" y1="137.16" x2="12.7" y2="137.16" width="0.1524" layer="91"/>
-<junction x="15.24" y="137.16"/>
-</segment>
 <segment>
 <wire x1="22.86" y1="63.5" x2="17.78" y2="63.5" width="0.1524" layer="91"/>
 <label x="17.78" y="63.5" size="1.27" layer="95" rot="R180" xref="yes"/>
 <pinref part="U3" gate="G$1" pin="A5"/>
+</segment>
+<segment>
+<pinref part="J1" gate="J1" pin="CAN-RX"/>
+<wire x1="17.78" y1="129.54" x2="15.24" y2="129.54" width="0.1524" layer="91"/>
+<label x="12.7" y="129.54" size="1.27" layer="95" rot="R180" xref="yes"/>
+<pinref part="TP1" gate="G$1" pin="1"/>
+<wire x1="15.24" y1="129.54" x2="12.7" y2="129.54" width="0.1524" layer="91"/>
+<wire x1="15.24" y1="129.54" x2="15.24" y2="132.08" width="0.1524" layer="91"/>
+<junction x="15.24" y="129.54"/>
 </segment>
 </net>
@@
 <segment>
 <pinref part="J1" gate="J1" pin="GND"/>
-<wire x1="17.78" y1="111.76" x2="15.24" y2="111.76" width="0.1524" layer="91"/>
-<wire x1="15.24" y1="111.76" x2="15.24" y2="109.22" width="0.1524" layer="91"/>
+<wire x1="17.78" y1="109.22" x2="15.24" y2="109.22" width="0.1524" layer="91"/>
+<wire x1="15.24" y1="109.22" x2="15.24" y2="106.68" width="0.1524" layer="91"/>
 <pinref part="GND1" gate="1" pin="GND"/>
 </segment>

Commit message: Housekeeping
Other:
- note added: "Nick P"
Changed lines of the file:
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@@
 <wire x1="226.06" y1="63.5" x2="226.06" y2="121.92" width="0.2032" layer="97" style="longdash"/>
 <text x="228.6" y="119.38" size="2.54" layer="97" align="top-left">CAN VCC LED</text>
+<text x="149.86" y="7.62" size="2.54" layer="94">Nick P</text>
 </plain>
 <instances>
